File: hw/sch_pcb/TFSBEC01A.kicad_sch (KiCad schematic)
At the start: 8 parts, among them J18 XT30PW-M, J19 XT30PW-F

Commit message: Edit
Parts:
- added J?: SM06B-GHS-TB, Connector_JST:JST_GH_SM06B-GHS-TB_1x06-1MP_P1.25mm_Horizontal, symbol MLAB_CONNECTORS_JST:SM06B-GHS-TB
- added J?: 505405-0670, Connector_JST:JST_GH_SM06B-GHS-TB_1x06-1MP_P1.25mm_Horizontal, symbol MLAB_CONNECTORS_JST:SM06B-GHS-TB
- added U?: ACS781LLRTR-050U-T, Sensor_Current:Allegro_PSOF-7_4.8x6.4mm_P1.60mm, symbol Sensor_Current:ACS781xLRTR-050U
Connections:
- net GND: now also J19.1 (-), U?.5 (IP+); no longer H1.1, H2.1, H3.1, H4.1
- net at J18.1 (-): now also U?.6 (IP-)
- net VCC: now reaches J18.2 (+)
- net VCC: now also J19.2 (+)
Other:
- moved on the sheet: J18, J19
Changed lines of the file:
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@@
   (page 1 1)
   (paper "A4")
-  (junction (at 259.08 22.86) (diameter 1.016) (color 0 0 0 0))
-  (junction (at 264.16 22.86) (diameter 1.016) (color 0 0 0 0))
-  (junction (at 267.97 22.86) (diameter 1.016) (color 0 0 0 0))
+  (junction (at 71.12 29.21) (diameter 1.016) (color 0 0 0 0))
+  (junction (at 71.12 34.29) (diameter 1.016) (color 0 0 0 0))
+  (wire (pts (xy 46.99 29.21) (xy 71.12 29.21))
+    (stroke (width 0) (type solid) (color 0 0 0 0))
+  )
+  (wire (pts (xy 46.99 34.29) (xy 54.61 34.29))
+    (stroke (width 0) (type solid) (color 0 0 0 0))
+  )
+  (wire (pts (xy 59.69 34.29) (xy 71.12 34.29))
+    (stroke (width 0) (type solid) (color 0 0 0 0))
+  )
+  (wire (pts (xy 71.12 27.94) (xy 71.12 29.21))
+    (stroke (width 0) (type solid) (color 0 0 0 0))
+  )
+  (wire (pts (xy 71.12 29.21) (xy 76.2 29.21))
+    (stroke (width 0) (type solid) (color 0 0 0 0))
+  )
+  (wire (pts (xy 71.12 34.29) (xy 71.12 35.56))
+    (stroke (width 0) (type solid) (color 0 0 0 0))
+  )
+  (wire (pts (xy 71.12 34.29) (xy 76.2 34.29))
+    (stroke (width 0) (type solid) (color 0 0 0 0))
+  )
   (wire (pts (xy 213.36 127) (xy 213.36 129.54))
     (stroke (width 0) (type solid) (color 0 0 0 0))
@@
     (stroke (width 0) (type solid) (color 0 0 0 0))
   )
-  (wire (pts (xy 250.19 22.86) (xy 259.08 22.86))
-    (stroke (width 0) (type solid) (color 0 0 0 0))
-  )
-  (wire (pts (xy 259.08 21.59) (xy 259.08 22.86))
-    (stroke (width 0) (type solid) (color 0 0 0 0))
-  )
-  (wire (pts (xy 259.08 22.86) (xy 264.16 22.86))
-    (stroke (width 0) (type solid) (color 0 0 0 0))
-  )
-  (wire (pts (xy 264.16 22.86) (xy 264.16 24.13))
-    (stroke (width 0) (type solid) (color 0 0 0 0))
-  )
-  (wire (pts (xy 264.16 22.86) (xy 267.97 22.86))
-    (stroke (width 0) (type solid) (color 0 0 0 0))
-  )
-  (wire (pts (xy 267.97 21.59) (xy 267.97 22.86))
-    (stroke (width 0) (type solid) (color 0 0 0 0))
-  )
-  (wire (pts (xy 267.97 22.86) (xy 275.59 22.86))
-    (stroke (width 0) (type solid) (color 0 0 0 0))
-  )
   (wire (pts (xy 275.59 22.86) (xy 275.59 21.59))
     (stroke (width 0) (type solid) (color 0 0 0 0))
+  )
+  (symbol (lib_id "power:VCC") (at 71.12 27.94 0) (unit 1)
+    (in_bom yes) (on_board yes)
+    (property "Reference" "#PWR?" (id 0) (at 71.12 31.75 0)
+      (effects (font (size 1.27 1.27)) hide)
+    )
+    (property "Value" "VCC" (id 1) (at 71.4883 23.6156 0))
+    (property "Footprint" "" (id 2) (at 71.12 27.94 0)
+      (effects (font (size 1.27 1.27)) hide)
+    )
+    (property "Datasheet" "" (id 3) (at 71.12 27.94 0)
+      (effects (font (size 1.27 1.27)) hide)
+    )
   )
   (symbol (lib_id "power:+5V") (at 213.36 127 0) (unit 1)
@@
     )
   )
-  (symbol (lib_id "power:GND") (at 264.16 24.13 0) (unit 1)
-    (in_bom yes) (on_board yes)
-    (property "Reference" "#PWR0121" (id 0) (at 264.16 30.48 0)
-      (effects (font (size 1.27 1.27)) hide)
-    )
-    (property "Value" "GND" (id 1) (at 264.2743 28.4544 0))
-    (property "Footprint" "" (id 2) (at 264.16 24.13 0)
-      (effects (font (size 1.27 1.27)) hide)
-    )
-    (property "Datasheet" "" (id 3) (at 264.16 24.13 0)
+  (symbol (lib_id "power:GND") (at 71.12 35.56 0) (unit 1)
+    (in_bom yes) (on_board yes)
+    (property "Reference" "#PWR?" (id 0) (at 71.12 41.91 0)
+      (effects (font (size 1.27 1.27)) hide)
+    )
+    (property "Value" "GND" (id 1) (at 71.2343 39.8844 0))
+    (property "Footprint" "" (id 2) (at 71.12 35.56 0)
+      (effects (font (size 1.27 1.27)) hide)
+    )
+    (property "Datasheet" "" (id 3) (at 71.12 35.56 0)
       (effects (font (size 1.27 1.27)) hide)
     )
@@
     )
   )
-  (symbol (lib_id "MLAB_CONNECTORS:XT30PW-F") (at 173.99 34.29 0) (mirror y) (unit 1)
-    (in_bom yes) (on_board yes)
-    (property "Reference" "J19" (id 0) (at 180.9751 33.0263 0)
-      (effects (font (size 1.27 1.27)) (justify right))
-    )
-    (property "Value" "XT30PW-F" (id 1) (at 180.9751 35.325 0)
-      (effects (font (size 1.27 1.27)) (justify right))
-    )
-    (property "Footprint" "Connector_AMASS:AMASS_XT30PW-F_1x02_P2.50mm_Horizontal" (id 2) (at 172.72 48.26 0)
-      (effects (font (size 1.27 1.27)) hide)
-    )
-    (property "Datasheet" "" (id 3) (at 173.99 30.48 0)
-      (effects (font (size 1.27 1.27)) hide)
-    )
-  )
-  (symbol (lib_id "MLAB_CONNECTORS:XT30PW-M") (at 127 34.29 0) (unit 1)
-    (in_bom yes) (on_board yes)
-    (property "Reference" "J18" (id 0) (at 125.2982 26.1682 0))
-    (property "Value" "XT30PW-M" (id 1) (at 125.2982 28.4669 0))
-    (property "Footprint" "Connector_AMASS:AMASS_XT30PW-M_1x02_P2.50mm_Horizontal" (id 2) (at 121.92 13.97 0)
-      (effects (font (size 1.27 1.27)) hide)
-    )
-    (property "Datasheet" "" (id 3) (at 121.92 13.97 0)
+  (symbol (lib_id "MLAB_CONNECTORS_JST:SM06B-GHS-TB") (at 220.98 66.04 0) (unit 1)
+    (in_bom yes) (on_board yes)
+    (property "Reference" "J?" (id 0) (at 222.8851 64.5719 0)
+      (effects (font (size 1.524 1.524)) (justify left))
+    )
+    (property "Value" " 505405-0670" (id 1) (at 222.885 67.28 0)
+      (effects (font (size 1.524 1.524)) (justify left))
+    )
+    (property "Footprint" "Connector_JST:JST_GH_SM06B-GHS-TB_1x06-1MP_P1.25mm_Horizontal" (id 2) (at 220.98 58.42 0)
+      (effects (font (size 1.524 1.524)) hide)
+    )
+    (property "Datasheet" "" (id 3) (at 220.98 58.42 0)
+      (effects (font (size 1.524 1.524)))
+    )
+  )
+  (symbol (lib_id "MLAB_CONNECTORS_JST:SM06B-GHS-TB") (at 220.98 90.17 0) (unit 1)
+    (in_bom yes) (on_board yes)
+    (property "Reference" "J?" (id 0) (at 222.8851 88.7019 0)
+      (effects (font (size 1.524 1.524)) (justify left))
+    )
+    (property "Value" "SM06B-GHS-TB" (id 1) (at 222.8851 91.4095 0)
+      (effects (font (size 1.524 1.524)) (justify left))
+    )
+    (property "Footprint" "Connector_JST:JST_GH_SM06B-GHS-TB_1x06-1MP_P1.25mm_Horizontal" (id 2) (at 220.98 82.55 0)
+      (effects (font (size 1.524 1.524)) hide)
+    )
+    (property "Datasheet" "" (id 3) (at 220.98 82.55 0)
+      (effects (font (size 1.524 1.524)))
+    )
+  )
+  (symbol (lib_id "MLAB_CONNECTORS:XT30PW-F") (at 85.09 31.75 0) (mirror y) (unit 1)
+    (in_bom yes) (on_board yes)
+    (property "Reference" "J19" (id 0) (at 92.0751 30.4863 0)
+      (effects (font (size 1.27 1.27)) (justify right))
+    )
+    (property "Value" "XT30PW-F" (id 1) (at 92.0751 32.785 0)
+      (effects (font (size 1.27 1.27)) (justify right))
+    )
+    (property "Footprint" "Connector_AMASS:AMASS_XT30PW-F_1x02_P2.50mm_Horizontal" (id 2) (at 83.82 45.72 0)
+      (effects (font (size 1.27 1.27)) hide)
+    )
+    (property "Datasheet" "" (id 3) (at 85.09 27.94 0)
+      (effects (font (size 1.27 1.27)) hide)
+    )
+  )
+  (symbol (lib_id "MLAB_CONNECTORS:XT30PW-M") (at 40.64 31.75 0) (unit 1)
+    (in_bom yes) (on_board yes)
+    (property "Reference" "J18" (id 0) (at 38.9382 23.6282 0))
+    (property "Value" "XT30PW-M" (id 1) (at 38.9382 25.9269 0))
+    (property "Footprint" "Connector_AMASS:AMASS_XT30PW-M_1x02_P2.50mm_Horizontal" (id 2) (at 35.56 11.43 0)
+      (effects (font (size 1.27 1.27)) hide)
+    )
+    (property "Datasheet" "" (id 3) (at 35.56 11.43 0)
+      (effects (font (size 1.27 1.27)) hide)
+    )
+  )
+  (symbol (lib_id "Sensor_Current:ACS781xLRTR-050U") (at 57.15 44.45 270) (unit 1)
+    (in_bom yes) (on_board yes)
+    (property "Reference" "U?" (id 0) (at 58.2994 55.6261 0)
+      (effects (font (size 1.27 1.27)) (justify left))
+    )
+    (property "Value" "ACS781LLRTR-050U-T" (id 1) (at 56.001 55.626 0)
+      (effects (font (size 1.27 1.27)) (justify left))
+    )
+    (property "Footprint" "Sensor_Current:Allegro_PSOF-7_4.8x6.4mm_P1.60mm" (id 2) (at 57.15 44.45 0)
+      (effects (font (size 1.27 1.27)) hide)
+    )
+    (property "Datasheet" "http://www.allegromicro.com/~/media/Files/Datasheets/ACS780-Datasheet.ashx?la=en" (id 3) (at 57.15 44.45 0)
       (effects (font (size 1.27 1.27)) hide)
     )
@@
       (reference "#PWR0119") (unit 1) (value "+5V") (footprint "")
     )
-    (path "/446f12bb-cc73-424f-ac32-7f06a17d5b9c"
-      (reference "#PWR0121") (unit 1) (value "GND") (footprint "")
+    (path "/74eb1aa0-7d99-4234-b011-2fd1f0a7fa77"
+      (reference "#PWR?") (unit 1) (value "GND") (footprint "")
+    )
+    (path "/7de54780-4207-4d5a-933d-460ab0bab915"
+      (reference "#PWR?") (unit 1) (value "VCC") (footprint "")
     )
     (path "/73f8190d-7547-4ed2-8230-76c4dc98b669"
@@
       (reference "J19") (unit 1) (value "XT30PW-F") (footprint "Connector_AMASS:AMASS_XT30PW-F_1x02_P2.50mm_Horizontal")
     )
+    (path "/f4d4d855-b613-4c7b-9018-a126dc8c8798"
+      (reference "J?") (unit 1) (value "SM06B-GHS-TB") (footprint "Connector_JST:JST_GH_SM06B-GHS-TB_1x06-1MP_P1.25mm_Horizontal")
+    )
+    (path "/f7f2aef6-4618-4662-b79f-b22f0cc5987f"
+      (reference "J?") (unit 1) (value " 505405-0670") (footprint "Connector_JST:JST_GH_SM06B-GHS-TB_1x06-1MP_P1.25mm_Horizontal")
+    )
     (path "/1d29942c-6664-43d9-a5ea-371615c39445"
       (reference "R3") (unit 1) (value "270R") (footprint "Mlab_R:SMD-0805")
     )
-  )
+    (path "/2c314da4-4c29-4f40-8ab0-280334610a81"
+      (reference "U?") (unit 1) (value "ACS781LLRTR-050U-T") (footprint "Sensor_Current:Allegro_PSOF-7_4.8x6.4mm_P1.60mm")
+    )
+  )
