File: hw/sch_pcb/TFSBEC01A.kicad_sch (KiCad schematic)
At the start: 11 parts, among them J18 XT30PW-M, J19 XT30PW-F

Commit message: Edit shema
Parts:
- removed D2: RED, Mlab_D:LED_1206, symbol Device:LED
- removed R3: 270R, Mlab_R:SMD-0805, symbol Device:R
- added C?: 100nF/50V, symbol Device:C
- added C? (x8): 10uF/50V, Resistor_SMD:R_1206_3216Metric, symbol Device:C
- added C? (x2): 100nF, Mlab_R:SMD-0603, symbol Device:C
- added C?: 22nF, symbol Device:C
- added C?: 1uF, Mlab_R:SMD-0805, symbol Device:C
- added C?: 10uF, Mlab_R:SMD-0805, symbol Device:C
- added C?: 1uF, Mlab_R:SMD-0603, symbol Device:C
- added C? (x2): 100uF/6V3, Resistor_SMD:R_1206_3216Metric, symbol Device:C
- added C?: 100nF, Mlab_R:SMD-0805, symbol Device:C
- added D?: PDS760-13, symbol Device:D_Schottky_AAK
- added D?: LED GREEN, Mlab_D:LED_1206, symbol Device:LED
- added D?: BZX585-B5V6.115, Diode_SMD:D_SOD-523, symbol MLAB_D:D_ZENER
- added L?: HCI1050-5R5, symbol Device:L
- added R?: 59kR, symbol Device:R
- added R?: 1k5, symbol Device:R
- added R?: 13k7, symbol Device:R
- added R? (x2): R, symbol Device:R
- added R?: 180R, Mlab_R:SMD-0603, symbol Device:R
- added U?: LMR14050, symbol MLAB_IO:LMR14050
- added U?: MIC5504-3.3YM5, Package_TO_SOT_SMD:SOT-23-5, symbol Regulator_Linear:MIC5504-3.3YM5
Connections:
- net GND: now also J?.5, J?.5, J?.6, J?.6, J?.MP, J?.MP, U?.2 (GND), C?.2, C?.2, C?.2, C?.2, C?.2, C?.2, C?.2, C?.2, C?.2, C?.2, C?.2, C?.2, C?.2, D?.1 (A), D?.1 (K), D?.2 (A), D?.2 (A), R?.2, R?.2, R?.2, U?.2 (GND), U?.7 (GND)
- net VCC: now also C?.1, C?.1, C?.1, C?.1, C?.1, C?.1, C?.1, C?.1, C?.1, R?.1, U?.2 (VIN), U?.3 (EN)
- net +3V3: now reaches U?.1 (VCC)
- net +3V3: now also C?.1, C?.1, U?.5 (VOUT)
- net SENSE_CURRENT: now reaches U?.3 (VOUT)
- net SENSE_CURRENT: now also J?.3, J?.3
- net 5V3: now reaches J?.1
- net 5V3: now also J?.1, J?.2, J?.2, C?.1, C?.1, C?.1, C?.1, C?.1, D?.1 (K), L?.2, R?.1, R?.1, U?.1 (VIN), U?.3 (EN)
- net SENSE_VOLTAGE: now reaches J?.4
- net SENSE_VOLTAGE: now also J?.4, R?.1, R?.2
- new net: R?.1, U?.4 (RT/SYNC)
- new net: C?.2, D?.3 (K), L?.1, U?.8 (SW)
- new net: C?.1, U?.6 (SS)
- new net: C?.1, U?.1 (BOOT)
- new net: R?.1, R?.2, U?.5 (FB)
- new net: D?.2 (A), R?.2
- no-connect marks 0 -> 2
Other:
- moved on the sheet: J?

Commit message: Edit
Parts:
- added C19: ?, Mlab_R:SMD-0805, symbol Device:C
- added R7: ?, Mlab_R:SMD-0805, symbol Device:R
- C12, C14: renamed from C?; footprint (none) -> Mlab_R:SMD-0805
- C13: renamed from C?; footprint Mlab_R:SMD-0603 -> Mlab_R:SMD-0805; UST_ID 5c70984812875079b91f8bc2 -> (none)
- C4, C5: renamed from C?; footprint Mlab_R:SMD-0603 -> Mlab_R:SMD-0805; UST_ID 5c70984812875079b91f8bf2 -> (none)
- D3: renamed from D?; footprint (none) -> Diode_SMD:D_PowerDI-5
- J1: renamed from J?; footprint Connector_JST:JST_GH_SM06B-GHS-TB_1x06-1MP_P1.25mm_Horizontal -> Connector_Molex:Molex_CLIK-Mate_505405-0670_1x06-1MP_P1.50mm_Vertical
- L1: renamed from L?; footprint (none) -> Inductor_SMD:L_Wuerth_HCI-1050
- R1: renamed from R?; footprint Mlab_R:SMD-0603 -> Mlab_R:SMD-0805
- R2, R3, R4, R5, R6: renamed from R?; footprint (none) -> Mlab_R:SMD-0805
- U3: renamed from U?; footprint (none) -> Package_SO:SOIC-8-1EP_3.9x4.9mm_P1.27mm_EP2.41x3.3mm_ThermalVias
- gave numbers to parts that had none: 18
Connections:
- net GND: now also C19.2
- net SENSE_CURRENT: now also C19.1, R7.2; no longer U1.3 (VOUT)
- new net: R7.1, U1.3 (VOUT)

Commit message: Edit PCB
Parts:
- removed D3: PDS760-13, Diode_SMD:D_PowerDI-5, symbol Device:D_Schottky_AAK
- added D3: PDS760-13, Diode_SMD:D_PowerDI-5, symbol Device:D_Schottky
- added D4: BZX585-B5V6.115, Diode_SMD:D_SOD-523, symbol MLAB_D:D_ZENER
- J1: value 505405-0670 -> 213226-0611
Connections:
- net GND: now also C11.2, C2.2, C7.2, C9.2, D3.2 (A), D4.2 (A)
- net SENSE_VOLTAGE: now also D4.1 (K)
- net at C15.2, L1.1, U3.8 (SW): now also D3.1 (K)
Changed lines of the file:
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@@
   (junction (at 102.87 86.36) (diameter 1.016) (color 0 0 0 0))
   (junction (at 107.95 41.91) (diameter 1.016) (color 0 0 0 0))
+  (junction (at 118.11 41.91) (diameter 1.016) (color 0 0 0 0))
   (junction (at 135.89 107.95) (diameter 1.016) (color 0 0 0 0))
-  (junction (at 135.89 118.11) (diameter 1.016) (color 0 0 0 0))
   (junction (at 157.48 107.95) (diameter 1.016) (color 0 0 0 0))
   (junction (at 167.64 107.95) (diameter 1.016) (color 0 0 0 0))
@@
     (stroke (width 0) (type solid) (color 0 0 0 0))
   )
+  (wire (pts (xy 25.4 115.57) (xy 25.4 116.84))
+    (stroke (width 0) (type solid) (color 0 0 0 0))
+  )
   (wire (pts (xy 31.75 173.99) (xy 31.75 175.26))
     (stroke (width 0) (type solid) (color 0 0 0 0))
@@
     (stroke (width 0) (type solid) (color 0 0 0 0))
   )
+  (wire (pts (xy 40.64 115.57) (xy 40.64 116.84))
+    (stroke (width 0) (type solid) (color 0 0 0 0))
+  )
   (wire (pts (xy 45.72 44.45) (xy 45.72 53.34))
     (stroke (width 0) (type solid) (color 0 0 0 0))
@@
     (stroke (width 0) (type solid) (color 0 0 0 0))
   )
+  (wire (pts (xy 54.61 115.57) (xy 54.61 116.84))
+    (stroke (width 0) (type solid) (color 0 0 0 0))
+  )
   (wire (pts (xy 55.88 180.34) (xy 55.88 175.26))
     (stroke (width 0) (type solid) (color 0 0 0 0))
@@
     (stroke (width 0) (type solid) (color 0 0 0 0))
   )
+  (wire (pts (xy 68.58 115.57) (xy 68.58 116.84))
+    (stroke (width 0) (type solid) (color 0 0 0 0))
+  )
   (wire (pts (xy 71.12 27.94) (xy 71.12 29.21))
     (stroke (width 0) (type solid) (color 0 0 0 0))
@@
     (stroke (width 0) (type solid) (color 0 0 0 0))
   )
-  (wire (pts (xy 107.95 41.91) (xy 114.3 41.91))
+  (wire (pts (xy 107.95 41.91) (xy 118.11 41.91))
     (stroke (width 0) (type solid) (color 0 0 0 0))
   )
@@
     (stroke (width 0) (type solid) (color 0 0 0 0))
   )
+  (wire (pts (xy 118.11 41.91) (xy 118.11 43.18))
+    (stroke (width 0) (type solid) (color 0 0 0 0))
+  )
+  (wire (pts (xy 118.11 41.91) (xy 123.19 41.91))
+    (stroke (width 0) (type solid) (color 0 0 0 0))
+  )
   (wire (pts (xy 123.19 101.6) (xy 125.73 101.6))
     (stroke (width 0) (type solid) (color 0 0 0 0))
@@
     (stroke (width 0) (type solid) (color 0 0 0 0))
   )
-  (wire (pts (xy 135.89 118.11) (xy 135.89 119.38))
-    (stroke (width 0) (type solid) (color 0 0 0 0))
-  )
-  (wire (pts (xy 135.89 118.11) (xy 138.43 118.11))
+  (wire (pts (xy 135.89 116.84) (xy 135.89 119.38))
     (stroke (width 0) (type solid) (color 0 0 0 0))
   )
@@
     (effects (font (size 1.27 1.27)) (justify left bottom))
   )
-  (label "SENSE_VOLTAGE" (at 114.3 41.91 0)
+  (label "SENSE_VOLTAGE" (at 123.19 41.91 0)
     (effects (font (size 1.27 1.27)) (justify left bottom))
   )
@@
     )
     (property "Datasheet" "" (id 3) (at 114.3 129.54 0)
+      (effects (font (size 1.27 1.27)) hide)
+    )
+    (pin "1")
+  )
+  (symbol (lib_id "power:GND") (at 118.11 53.34 0) (unit 1)
+    (in_bom yes) (on_board yes)
+    (property "Reference" "#PWR0135" (id 0) (at 118.11 59.69 0)
+      (effects (font (size 1.27 1.27)) hide)
+    )
+    (property "Value" "GND" (id 1) (at 118.2243 57.6644 0))
+    (property "Footprint" "" (id 2) (at 118.11 53.34 0)
+      (effects (font (size 1.27 1.27)) hide)
+    )
+    (property "Datasheet" "" (id 3) (at 118.11 53.34 0)
       (effects (font (size 1.27 1.27)) hide)
     )
@@
     (pin "1")
   )
+  (symbol (lib_id "Device:D_Schottky") (at 135.89 113.03 270) (unit 1)
+    (in_bom yes) (on_board yes) (fields_autoplaced)
+    (property "Reference" "D3" (id 0) (at 137.9221 112.2691 90)
+      (effects (font (size 1.27 1.27)) (justify left))
+    )
+    (property "Value" "PDS760-13" (id 1) (at 137.9221 114.5678 90)
+      (effects (font (size 1.27 1.27)) (justify left))
+    )
+    (property "Footprint" "Diode_SMD:D_PowerDI-5" (id 2) (at 135.89 113.03 0)
+      (effects (font (size 1.27 1.27)) hide)
+    )
+    (property "Datasheet" "~" (id 3) (at 135.89 113.03 0)
+      (effects (font (size 1.27 1.27)) hide)
+    )
+    (pin "1")
+    (pin "2")
+  )
   (symbol (lib_id "MLAB_D:D_ZENER") (at 46.99 181.61 270) (unit 1)
     (in_bom yes) (on_board yes)
@@
     )
     (property "UST_ID" "604b0326128750769e5b0f93" (id 5) (at 46.99 181.61 0)
+      (effects (font (size 1.27 1.27)) hide)
+    )
+    (pin "1")
+    (pin "2")
+  )
+  (symbol (lib_id "MLAB_D:D_ZENER") (at 118.11 48.26 270) (unit 1)
+    (in_bom yes) (on_board yes)
+    (property "Reference" "D4" (id 0) (at 120.1166 47.0916 90)
+      (effects (font (size 1.27 1.27)) (justify left))
+    )
+    (property "Value" "BZX585-B5V6.115" (id 1) (at 120.117 51.943 90)
+      (effects (font (size 1.27 1.27)) (justify left))
+    )
+    (property "Footprint" "Diode_SMD:D_SOD-523" (id 2) (at 118.11 48.26 0)
+      (effects (font (size 1.524 1.524)) hide)
+    )
+    (property "Datasheet" "" (id 3) (at 118.11 48.26 0)
+      (effects (font (size 1.524 1.524)))
+    )
+    (property "UST_id" "" (id 4) (at 118.11 48.26 0)
+      (effects (font (size 1.27 1.27)) hide)
+    )
+    (property "UST_ID" "604b0326128750769e5b0f93" (id 5) (at 118.11 48.26 0)
       (effects (font (size 1.27 1.27)) hide)
     )
@@
     (pin "2")
   )
-  (symbol (lib_id "Device:D_Schottky_AAK") (at 135.89 113.03 270) (unit 1)
-    (in_bom yes) (on_board yes) (fields_autoplaced)
-    (property "Reference" "D3" (id 0) (at 139.4461 112.9041 90)
-      (effects (font (size 1.27 1.27)) (justify left))
-    )
-    (property "Value" "PDS760-13" (id 1) (at 139.4461 115.2028 90)
-      (effects (font (size 1.27 1.27)) (justify left))
-    )
-    (property "Footprint" "Diode_SMD:D_PowerDI-5" (id 2) (at 135.89 113.03 0)
-      (effects (font (size 1.27 1.27)) hide)
-    )
-    (property "Datasheet" "~" (id 3) (at 135.89 113.03 0)
-      (effects (font (size 1.27 1.27)) hide)
-    )
-    (pin "1")
-    (pin "2")
-    (pin "3")
-  )
   (symbol (lib_id "MLAB_CONNECTORS:XT30PW-F") (at 85.09 31.75 0) (mirror y) (unit 1)
     (in_bom yes) (on_board yes)
@@
       (effects (font (size 1.524 1.524)) (justify left))
     )
-    (property "Value" " 505405-0670" (id 1) (at 260.985 49.5 0)
+    (property "Value" "213226-0611" (id 1) (at 260.985 49.5 0)
       (effects (font (size 1.524 1.524)) (justify left))
     )
@@
       (reference "#PWR0134") (unit 1) (value "GND") (footprint "")
     )
+    (path "/689bc101-b676-4846-9f31-475fea18647f"
+      (reference "#PWR0135") (unit 1) (value "GND") (footprint "")
+    )
     (path "/77a04708-d7dd-4038-877a-2a70cb335565"
       (reference "C1") (unit 1) (value "10uF/50V") (footprint "Resistor_SMD:R_1206_3216Metric")
@@
       (reference "D2") (unit 1) (value "BZX585-B5V6.115") (footprint "Diode_SMD:D_SOD-523")
     )
-    (path "/204c49b6-664f-4a7d-82bd-1838d905780f"
+    (path "/b25ff9ae-55ba-49fe-8fc3-f9a989d7233e"
       (reference "D3") (unit 1) (value "PDS760-13") (footprint "Diode_SMD:D_PowerDI-5")
+    )
+    (path "/70024b90-f1b2-428f-87e4-7b38c6bdbb16"
+      (reference "D4") (unit 1) (value "BZX585-B5V6.115") (footprint "Diode_SMD:D_SOD-523")
     )
     (path "/9ccdf6af-8340-4776-9e1b-cf90430c2f74"
@@
     )
     (path "/f7f2aef6-4618-4662-b79f-b22f0cc5987f"
-      (reference "J1") (unit 1) (value " 505405-0670") (footprint "Connector_Molex:Molex_CLIK-Mate_505405-0670_1x06-1MP_P1.50mm_Vertical")
+      (reference "J1") (unit 1) (value "213226-0611") (footprint "Connector_Molex:Molex_CLIK-Mate_505405-0670_1x06-1MP_P1.50mm_Vertical")
     )
     (path "/f4d4d855-b613-4c7b-9018-a126dc8c8798"

Commit message: Edit PCB
Parts:
- removed H1, H2, H3, H4: M3, Mlab_Mechanical:MountingHole_3mm, symbol Mechanical:MountingHole_Pad
Connections:
- net 5V3: now also J1.5, J1.6; no longer J1.1, J1.2
- net GND: now also J1.1, J1.2, U3.9 (GND); no longer J1.5, J1.6
- net SENSE_CURRENT: now also J1.4; no longer J1.3
- net SENSE_VOLTAGE: now also J1.3; no longer J1.4
Changed lines of the file:
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@@
   (junction (at 204.47 127) (diameter 1.016) (color 0 0 0 0))
   (junction (at 250.19 40.64) (diameter 1.016) (color 0 0 0 0))
-  (junction (at 250.19 53.34) (diameter 1.016) (color 0 0 0 0))
-  (junction (at 250.19 55.88) (diameter 1.016) (color 0 0 0 0))
+  (junction (at 250.19 50.8) (diameter 1.016) (color 0 0 0 0))
   (junction (at 250.19 74.93) (diameter 1.016) (color 0 0 0 0))
   (junction (at 250.19 87.63) (diameter 1.016) (color 0 0 0 0))
@@
     (stroke (width 0) (type solid) (color 0 0 0 0))
   )
+  (wire (pts (xy 245.11 36.83) (xy 250.19 36.83))
+    (stroke (width 0) (type solid) (color 0 0 0 0))
+  )
+  (wire (pts (xy 247.65 50.8) (xy 250.19 50.8))
+    (stroke (width 0) (type solid) (color 0 0 0 0))
+  )
   (wire (pts (xy 248.92 45.72) (xy 254 45.72))
     (stroke (width 0) (type solid) (color 0 0 0 0))
@@
     (stroke (width 0) (type solid) (color 0 0 0 0))
   )
-  (wire (pts (xy 250.19 21.59) (xy 250.19 22.86))
-    (stroke (width 0) (type solid) (color 0 0 0 0))
-  )
   (wire (pts (xy 250.19 36.83) (xy 250.19 40.64))
     (stroke (width 0) (type solid) (color 0 0 0 0))
@@
     (stroke (width 0) (type solid) (color 0 0 0 0))
   )
-  (wire (pts (xy 250.19 53.34) (xy 250.19 55.88))
-    (stroke (width 0) (type solid) (color 0 0 0 0))
-  )
   (wire (pts (xy 250.19 55.88) (xy 250.19 58.42))
     (stroke (width 0) (type solid) (color 0 0 0 0))
@@
   )
   (wire (pts (xy 254 87.63) (xy 250.19 87.63))
-    (stroke (width 0) (type solid) (color 0 0 0 0))
-  )
-  (wire (pts (xy 275.59 22.86) (xy 275.59 21.59))
     (stroke (width 0) (type solid) (color 0 0 0 0))
   )
@@
     (effects (font (size 1.27 1.27)) (justify right bottom))
   )
-  (label "SENSE_CURRENT" (at 248.92 45.72 180)
+  (label "5V3" (at 247.65 50.8 180)
     (effects (font (size 1.27 1.27)) (justify right bottom))
   )
-  (label "SENSE_VOLTAGE" (at 248.92 48.26 180)
+  (label "SENSE_VOLTAGE" (at 248.92 45.72 180)
+    (effects (font (size 1.27 1.27)) (justify right bottom))
+  )
+  (label "SENSE_CURRENT" (at 248.92 48.26 180)
     (effects (font (size 1.27 1.27)) (justify right bottom))
   )
@@
     (effects (font (size 1.27 1.27)) (justify right bottom))
   )
-  (label "5V3" (at 250.19 36.83 180)
-    (effects (font (size 1.27 1.27)) (justify right bottom))
-  )
   (label "5V3" (at 250.19 71.12 180)
     (effects (font (size 1.27 1.27)) (justify right bottom))
@@
     )
     (property "Datasheet" "" (id 3) (at 204.47 137.16 0)
+      (effects (font (size 1.27 1.27)) hide)
+    )
+    (pin "1")
+  )
+  (symbol (lib_id "power:GND") (at 245.11 36.83 0) (unit 1)
+    (in_bom yes) (on_board yes)
+    (property "Reference" "#PWR0136" (id 0) (at 245.11 43.18 0)
+      (effects (font (size 1.27 1.27)) hide)
+    )
+    (property "Value" "GND" (id 1) (at 245.2243 41.1544 0))
+    (property "Footprint" "" (id 2) (at 245.11 36.83 0)
+      (effects (font (size 1.27 1.27)) hide)
+    )
+    (property "Datasheet" "" (id 3) (at 245.11 36.83 0)
       (effects (font (size 1.27 1.27)) hide)
     )
@@
     (pin "1")
     (pin "2")
-  )
-  (symbol (lib_id "Mechanical:MountingHole_Pad") (at 250.19 19.05 0) (unit 1)
-    (in_bom yes) (on_board yes)
-    (property "Reference" "H1" (id 0) (at 252.7301 17.7736 0)
-      (effects (font (size 1.27 1.27)) (justify left))
-    )
-    (property "Value" "M3" (id 1) (at 252.7301 20.0723 0)
-      (effects (font (size 1.27 1.27)) (justify left))
-    )
-    (property "Footprint" "Mlab_Mechanical:MountingHole_3mm" (id 2) (at 250.19 19.05 0)
-      (effects (font (size 1.27 1.27)) hide)
-    )
-    (property "Datasheet" "~" (id 3) (at 250.19 19.05 0)
-      (effects (font (size 1.27 1.27)) hide)
-    )
-    (pin "1")
-  )
-  (symbol (lib_id "Mechanical:MountingHole_Pad") (at 259.08 19.05 0) (unit 1)
-    (in_bom yes) (on_board yes)
-    (property "Reference" "H2" (id 0) (at 261.6201 17.7736 0)
-      (effects (font (size 1.27 1.27)) (justify left))
-    )
-    (property "Value" "M3" (id 1) (at 261.6201 20.0723 0)
-      (effects (font (size 1.27 1.27)) (justify left))
-    )
-    (property "Footprint" "Mlab_Mechanical:MountingHole_3mm" (id 2) (at 259.08 19.05 0)
-      (effects (font (size 1.27 1.27)) hide)
-    )
-    (property "Datasheet" "~" (id 3) (at 259.08 19.05 0)
-      (effects (font (size 1.27 1.27)) hide)
-    )
-    (pin "1")
-  )
-  (symbol (lib_id "Mechanical:MountingHole_Pad") (at 267.97 19.05 0) (unit 1)
-    (in_bom yes) (on_board yes)
-    (property "Reference" "H3" (id 0) (at 270.5101 17.7736 0)
-      (effects (font (size 1.27 1.27)) (justify left))
-    )
-    (property "Value" "M3" (id 1) (at 270.5101 20.0723 0)
-      (effects (font (size 1.27 1.27)) (justify left))
-    )
-    (property "Footprint" "Mlab_Mechanical:MountingHole_3mm" (id 2) (at 267.97 19.05 0)
-      (effects (font (size 1.27 1.27)) hide)
-    )
-    (property "Datasheet" "~" (id 3) (at 267.97 19.05 0)
-      (effects (font (size 1.27 1.27)) hide)
-    )
-    (pin "1")
-  )
-  (symbol (lib_id "Mechanical:MountingHole_Pad") (at 275.59 19.05 0) (unit 1)
-    (in_bom yes) (on_board yes)
-    (property "Reference" "H4" (id 0) (at 278.1301 17.7736 0)
-      (effects (font (size 1.27 1.27)) (justify left))
-    )
-    (property "Value" "M3" (id 1) (at 278.1301 20.0723 0)
-      (effects (font (size 1.27 1.27)) (justify left))
-    )
-    (property "Footprint" "Mlab_Mechanical:MountingHole_3mm" (id 2) (at 275.59 19.05 0)
-      (effects (font (size 1.27 1.27)) hide)
-    )
-    (property "Datasheet" "~" (id 3) (at 275.59 19.05 0)
-      (effects (font (size 1.27 1.27)) hide)
-    )
-    (pin "1")
   )
   (symbol (lib_id "Device:D_Schottky") (at 135.89 113.03 270) (unit 1)
@@
     (pin "7")
     (pin "8")
+    (pin "9")
   )
   (sheet_instances
@@
       (reference "#PWR0135") (unit 1) (value "GND") (footprint "")
     )
+    (path "/5c1b09e4-3480-4819-a63d-0146ed13b776"
+      (reference "#PWR0136") (unit 1) (value "GND") (footprint "")
+    )
     (path "/77a04708-d7dd-4038-877a-2a70cb335565"
       (reference "C1") (unit 1) (value "10uF/50V") (footprint "Resistor_SMD:R_1206_3216Metric")
@@
       (reference "D4") (unit 1) (value "BZX585-B5V6.115") (footprint "Diode_SMD:D_SOD-523")
     )
-    (path "/9ccdf6af-8340-4776-9e1b-cf90430c2f74"
-      (reference "H1") (unit 1) (value "M3") (footprint "Mlab_Mechanical:MountingHole_3mm")
-    )
-    (path "/d5b4ee16-e759-497e-8377-97158519928e"
-      (reference "H2") (unit 1) (value "M3") (footprint "Mlab_Mechanical:MountingHole_3mm")
-    )
-    (path "/760863e4-da73-4058-a60b-a7063f12c80c"
-      (reference "H3") (unit 1) (value "M3") (footprint "Mlab_Mechanical:MountingHole_3mm")
-    )
-    (path "/6c86aaaa-9174-4bc6-95df-e076880a11e1"
-      (reference "H4") (unit 1) (value "M3") (footprint "Mlab_Mechanical:MountingHole_3mm")
-    )
     (path "/f7f2aef6-4618-4662-b79f-b22f0cc5987f"
