File: hw/sch_pcb/TFSBEC01A.kicad_sch (KiCad schematic)
At the start: 38 parts, among them J1 213226-0611, J18 XT30PW-M, J19 XT30PW-F, J2 SM06B-GHS-TB, U1 ACS781LLRTR-050U-T, U2 MIC5504-3.3YM5, U3 LMR14050

Commit message: Edit
Parts:
- C13: UST_ID (none) -> 5c70984712875079b91f8b50
- C14: UST_ID (none) -> 5c70984712875079b91f8b4a
- C15, C4, C5: UST_ID (none) -> 5c70984712875079b91f8b4c
- C19: value ? -> 22nF; UST_ID (none) -> 5c70984712875079b91f8b4a
- D1: UST_ID (none) -> 5c70984412875079b91f8895
- D2, D4: UST_ID 604b0326128750769e5b0f93 -> 60879d38128750769ee58e48
- D3: UST_ID (none) -> 6087aaaf128750769ee58fb7
- J1: UST_ID (none) -> 6087ab22128750769ee58ff1
- J18: UST_ID (none) -> 5c70984812875079b91f8ba8
- J19: UST_ID (none) -> 6087ae38128750769ee59039
- J2: UST_ID (none) -> 5fa0f70212875025b3977932
- L1: UST_ID (none) -> 6087af42128750769ee59060
- R1: UST_ID (none) -> 5c70984512875079b91f897c
- R2: UST_ID (none) -> 6087b414128750769ee590a1
- R3: UST_ID (none) -> 6087b4ba128750769ee590cd
- R4: UST_ID (none) -> 5c70984512875079b91f898e
- R5: value R -> 91k; UST_ID (none) -> 5c70984712875079b91f8a95
- R6: value R -> 15k; UST_ID (none) -> 5c70984712875079b91f8b6a
- R7: value ? -> 1k5; UST_ID (none) -> 5c70984512875079b91f898e
- U1: UST_ID (none) -> 6087b619128750769ee590fa
- U3: UST_ID (none) -> 6087b6ba128750769ee59110
Changed lines of the file:
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@@
+      (effects (font (size 1.27 1.27)) hide)
+    )
+    (property "UST_ID" "6087af42128750769ee59060" (id 4) (at 146.05 107.95 0)
       (effects (font (size 1.27 1.27)) hide)
     )
@@
       (effects (font (size 1.27 1.27)) hide)
     )
+    (property "UST_ID" "5c70984512875079b91f897c" (id 4) (at 24.13 175.26 0)
+      (effects (font (size 1.27 1.27)) hide)
+    )
     (pin "1")
     (pin "2")
@@
     (in_bom yes) (on_board yes) (fields_autoplaced)
     (property "Reference" "R7" (id 0) (at 68.58 52.7008 90))
-    (property "Value" "?" (id 1) (at 68.58 54.9995 90))
+    (property "Value" "1k5" (id 1) (at 68.58 54.9995 90))
     (property "Footprint" "Mlab_R:SMD-0805" (id 2) (at 68.58 58.928 90)
       (effects (font (size 1.27 1.27)) hide)
@@
       (effects (font (size 1.27 1.27)) hide)
     )
+    (property "UST_ID" "5c70984512875079b91f898e" (id 4) (at 68.58 57.15 0)
+      (effects (font (size 1.27 1.27)) hide)
+    )
     (pin "1")
     (pin "2")
@@
       (effects (font (size 1.27 1.27)) hide)
     )
+    (property "UST_ID" "6087b414128750769ee590a1" (id 4) (at 90.17 124.46 0)
+      (effects (font (size 1.27 1.27)) hide)
+    )
     (pin "1")
     (pin "2")
@@
       (effects (font (size 1.27 1.27)) hide)
     )
+    (property "UST_ID" "6087b4ba128750769ee590cd" (id 4) (at 107.95 36.83 0)
+      (effects (font (size 1.27 1.27)) hide)
+    )
     (pin "1")
     (pin "2")
@@
       (effects (font (size 1.27 1.27)) hide)
     )
+    (property "UST_ID" "5c70984512875079b91f898e" (id 4) (at 107.95 46.99 0)
+      (effects (font (size 1.27 1.27)) hide)
+    )
     (pin "1")
     (pin "2")
@@
       (effects (font (size 1.27 1.27)) (justify left))
     )
-    (property "Value" "R" (id 1) (at 206.2481 123.4578 0)
+    (property "Value" "91k" (id 1) (at 206.2481 123.4578 0)
       (effects (font (size 1.27 1.27)) (justify left))
     )
@@
       (effects (font (size 1.27 1.27)) hide)
     )
+    (property "UST_ID" "5c70984712875079b91f8a95" (id 4) (at 204.47 121.92 0)
+      (effects (font (size 1.27 1.27)) hide)
+    )
     (pin "1")
     (pin "2")
@@
       (effects (font (size 1.27 1.27)) (justify left))
     )
-    (property "Value" "R" (id 1) (at 206.2481 133.6178 0)
+    (property "Value" "15k" (id 1) (at 206.2481 133.6178 0)
       (effects (font (size 1.27 1.27)) (justify left))
     )
@@
       (effects (font (size 1.27 1.27)) hide)
     )
+    (property "UST_ID" "5c70984712875079b91f8b6a" (id 4) (at 204.47 132.08 0)
+      (effects (font (size 1.27 1.27)) hide)
+    )
     (pin "1")
     (pin "2")
@@
     )
     (property "Datasheet" "~" (id 3) (at 135.89 113.03 0)
+      (effects (font (size 1.27 1.27)) hide)
+    )
+    (property "UST_ID" "6087aaaf128750769ee58fb7" (id 4) (at 135.89 113.03 0)
       (effects (font (size 1.27 1.27)) hide)
     )
@@
       (effects (font (size 1.27 1.27)) hide)
     )
-    (property "UST_ID" "604b0326128750769e5b0f93" (id 5) (at 46.99 181.61 0)
+    (property "UST_ID" "60879d38128750769ee58e48" (id 5) (at 46.99 181.61 0)
       (effects (font (size 1.27 1.27)) hide)
     )
@@
       (effects (font (size 1.27 1.27)) hide)
     )
-    (property "UST_ID" "604b0326128750769e5b0f93" (id 5) (at 118.11 48.26 0)
+    (property "UST_ID" "60879d38128750769ee58e48" (id 5) (at 118.11 48.26 0)
       (effects (font (size 1.27 1.27)) hide)
     )
@@
       (effects (font (size 1.27 1.27)) hide)
     )
+    (property "UST_ID" "5c70984412875079b91f8895" (id 4) (at 24.13 184.15 0)
+      (effects (font (size 1.27 1.27)) hide)
+    )
     (pin "1")
     (pin "2")
@@
       (effects (font (size 1.27 1.27)) hide)
     )
-    (property "UST_ID" "" (id 5) (at 35.56 48.26 0)
+    (property "UST_ID" "5c70984712875079b91f8b4c" (id 5) (at 35.56 48.26 0)
       (effects (font (size 1.27 1.27)) hide)
     )
@@
       (effects (font (size 1.27 1.27)) hide)
     )
-    (property "UST_ID" "" (id 5) (at 39.37 181.61 0)
+    (property "UST_ID" "5c70984712875079b91f8b4c" (id 5) (at 39.37 181.61 0)
       (effects (font (size 1.27 1.27)) hide)
     )
@@
       (effects (font (size 1.27 1.27)) (justify left))
     )
-    (property "Value" "?" (id 1) (at 79.1211 63.7678 0)
+    (property "Value" "22nF" (id 1) (at 79.1211 63.7678 0)
       (effects (font (size 1.27 1.27)) (justify left))
     )
@@
       (effects (font (size 1.27 1.27)) hide)
     )
-    (property "UST_ID" "" (id 4) (at 76.2 62.23 0)
+    (property "UST_ID" "5c70984712875079b91f8b4a" (id 4) (at 76.2 62.23 0)
       (effects (font (size 1.27 1.27)) hide)
     )
@@
       (effects (font (size 1.27 1.27)) hide)
     )
-    (property "UST_ID" "" (id 5) (at 85.09 181.61 0)
+    (property "UST_ID" "5c70984712875079b91f8b50" (id 5) (at 85.09 181.61 0)
       (effects (font (size 1.27 1.27)) hide)
     )
@@
     )
     (property "Datasheet" "~" (id 3) (at 99.06 124.46 0)
+      (effects (font (size 1.27 1.27)) hide)
+    )
+    (property "UST_ID" "5c70984712875079b91f8b4a" (id 4) (at 99.06 124.46 0)
       (effects (font (size 1.27 1.27)) hide)
     )
@@
       (effects (font (size 1.27 1.27)) hide)
     )
-    (property "Datasheet" "~" (id 3) (at 129.54 101.6 0)
+    (property "Datasheet" "" (id 3) (at 129.54 101.6 0)
+      (effects (font (size 1.27 1.27)) hide)
+    )
+    (property "UST_ID" "5c70984712875079b91f8b4c" (id 4) (at 129.54 101.6 0)
       (effects (font (size 1.27 1.27)) hide)
     )
@@
       (effects (font (size 1.27 1.27)) hide)
     )
+    (property "UST_ID" "6087ae38128750769ee59039" (id 4) (at 85.09 31.75 0)
+      (effects (font (size 1.27 1.27)) hide)
+    )
     (pin "1")
     (pin "2")
@@
     (property "Datasheet" "" (id 3) (at 259.08 40.64 0)
       (effects (font (size 1.524 1.524)))
+    )
+    (property "UST_ID" "6087ab22128750769ee58ff1" (id 4) (at 259.08 48.26 0)
+      (effects (font (size 1.27 1.27)) hide)
     )
     (pin "1")
@@
       (effects (font (size 1.524 1.524)))
     )
+    (property "UST_ID" "5fa0f70212875025b3977932" (id 4) (at 259.08 82.55 0)
+      (effects (font (size 1.27 1.27)) hide)
+    )
     (pin "1")
     (pin "2")
@@
       (effects (font (size 1.27 1.27)) hide)
     )
+    (property "UST_ID" "5c70984812875079b91f8ba8" (id 4) (at 40.64 31.75 0)
+      (effects (font (size 1.27 1.27)) hide)
+    )
     (pin "1")
     (pin "2")
@@
     )
     (property "Datasheet" "http://www.allegromicro.com/~/media/Files/Datasheets/ACS780-Datasheet.ashx?la=en" (id 3) (at 57.15 44.45 0)
+      (effects (font (size 1.27 1.27)) hide)
+    )
+    (property "UST_ID" "6087b619128750769ee590fa" (id 4) (at 57.15 44.45 0)
       (effects (font (size 1.27 1.27)) hide)
     )
@@
     )
     (property "Datasheet" "" (id 3) (at 114.3 113.03 0)
+      (effects (font (size 1.27 1.27)) hide)
+    )
+    (property "UST_ID" "6087b6ba128750769ee59110" (id 4) (at 114.3 113.03 0)
       (effects (font (size 1.27 1.27)) hide)
     )
@@
     )
     (path "/83999c1d-9f92-4e73-9899-cd35a6e55aaf"
-      (reference "C19") (unit 1) (value "?") (footprint "Mlab_R:SMD-0805")
+      (reference "C19") (unit 1) (value "22nF") (footprint "Mlab_R:SMD-0805")
     )
     (path "/a10f1d61-be74-44c2-a2c9-0fc5f6ad4197"
@@
     )
     (path "/aca61bab-0b2d-4525-a700-8f1144afeab3"
-      (reference "R5") (unit 1) (value "R") (footprint "Mlab_R:SMD-0805")
+      (reference "R5") (unit 1) (value "91k") (footprint "Mlab_R:SMD-0805")
     )
     (path "/8188ab8e-ba48-48c3-8771-5459014c4f14"
-      (reference "R6") (unit 1) (value "R") (footprint "Mlab_R:SMD-0805")
+      (reference "R6") (unit 1) (value "15k") (footprint "Mlab_R:SMD-0805")
     )
     (path "/1b698215-853e-4e3d-a0e4-baa678b4255c"
-      (reference "R7") (unit 1) (value "?") (footprint "Mlab_R:SMD-0805")
+      (reference "R7") (unit 1) (value "1k5") (footprint "Mlab_R:SMD-0805")
     )
     (path "/2c314da4-4c29-4f40-8ab0-280334610a81"

Commit message: Update project to KiCAD 6.0. Update title block.
Other:
- company: (none) -> ThunderFly s.r.o.
- title: (none) -> TFSBEC01A
