File: hw/sch_pcb/TFSBEC01A.kicad_pcb (KiCad board)
At the start: 2 copper layers, 40.1 x 30 mm, 7 parts, among them J18 XT30PW-M, J19 XT30PW-F

Commit message: Edit
Parts:
- added C1: 10uF/50V, Resistor_SMD:R_1206_3216Metric, F.Cu at (66.2, -32.6)
- added C10: 10uF/50V, Resistor_SMD:R_1206_3216Metric, F.Cu at (85.8, -41.3)
- added C11: 10uF/50V, Resistor_SMD:R_1206_3216Metric, F.Cu at (80.2, -41.3)
- added C12: 100nF/50V, Mlab_R:SMD-0805, F.Cu at (80.9, -35.0)
- added C13: 1uF, Mlab_R:SMD-0805, F.Cu at (85.1, -35.6)
- added C14: 22nF, Mlab_R:SMD-0805, F.Cu at (77.7, -32.3)
- added C15: 100nF, Mlab_R:SMD-0805, F.Cu at (95.6, -49.6)
- added C16: 1uF, Mlab_R:SMD-0805, F.Cu at (72.9, -25.0)
- added C17: 100uF/6V3, Resistor_SMD:R_1206_3216Metric, F.Cu at (68.0, -29.3)
- added C18: 100uF/6V3, Resistor_SMD:R_1206_3216Metric, F.Cu at (90.7, -49.3)
- added C19: ?, Mlab_R:SMD-0805, F.Cu at (75.1, -22.0)
- added C2: 10uF/50V, Resistor_SMD:R_1206_3216Metric, F.Cu at (71.8, -32.6)
- added C3: 10uF, Mlab_R:SMD-0805, F.Cu at (81.9, -32.3)
- added C4: 100nF, Mlab_R:SMD-0805, F.Cu at (77.7, -29.6)
- added C5: 100nF, Mlab_R:SMD-0805, F.Cu at (90.7, -43.7)
- added C6: 10uF/50V, Resistor_SMD:R_1206_3216Metric, F.Cu at (68.0, -26.1)
- added C7: 10uF/50V, Resistor_SMD:R_1206_3216Metric, F.Cu at (74.6, -41.9)
- added C8: 10uF/50V, Resistor_SMD:R_1206_3216Metric, F.Cu at (74.6, -38.6)
- added C9: 10uF/50V, Resistor_SMD:R_1206_3216Metric, F.Cu at (80.2, -38.0)
- added D1: LED GREEN, Mlab_D:LED_1206, F.Cu at (62.1, -27.0)
- added D2: BZX585-B5V6.115, Diode_SMD:D_SOD-523, F.Cu at (89.0, -38.4)
- added D3: PDS760-13, Diode_SMD:D_PowerDI-5, F.Cu at (54.7, -26.2)
- added J1: 505405-0670, Connector_Molex:Molex_CLIK-Mate_505405-0670_1x06-1MP_P1.50mm_Vertical, F.Cu at (86.4, -25.0)
- added J2: SM06B-GHS-TB, Connector_JST:JST_GH_SM06B-GHS-TB_1x06-1MP_P1.25mm_Horizontal, F.Cu at (74.2, -51.8)
- added L1: HCI1050-5R5, Inductor_SMD:L_Wuerth_HCI-1050, F.Cu at (56.8, -34.9)
- added R1: 180R, Mlab_R:SMD-0805, F.Cu at (95.6, -46.9)
- added R2: 59kR, Mlab_R:SMD-0805, F.Cu at (90.7, -41.0)
- added R3: 13k7, Mlab_R:SMD-0805, F.Cu at (90.0, -46.3)
- added R4: 1k5, Mlab_R:SMD-0805, F.Cu at (76.7, -35.0)
- added R5: R, Mlab_R:SMD-0805, F.Cu at (85.1, -38.3)
- added R6: R, Mlab_R:SMD-0805, F.Cu at (69.0, -42.2)
- added R7: ?, Mlab_R:SMD-0805, F.Cu at (70.9, -22.0)
- added U1: ACS781LLRTR-050U-T, Sensor_Current:Allegro_PSOF-7_4.8x6.4mm_P1.60mm, F.Cu at (83.9, -46.9)
- added U2: MIC5504-3.3YM5, Package_TO_SOT_SMD:SOT-23-5, F.Cu at (73.2, -28.7)
- added U3: LMR14050, Package_SO:SOIC-8-1EP_3.9x4.9mm_P1.27mm_EP2.41x3.3mm_ThermalVias, F.Cu at (96.8, -27.7)
- moved J19 95.0 mm to (100.3, -35.3)
- moved J18 38.6 mm to (62.8, -50.9), turned to 90 degrees
Connections:
- H1 pad 1: GND -> unconnected-(H1-Pad1)
- H2 pad 1: GND -> unconnected-(H2-Pad1)
- H3 pad 1: GND -> unconnected-(H3-Pad1)
- H4 pad 1: GND -> unconnected-(H4-Pad1)
- J18 pad 1: (no net) -> Net-(J18-Pad1)
- J18 pad 2: (no net) -> VCC
- J19 pad 1: (no net) -> GND
- J19 pad 2: (no net) -> VCC

Commit message: Edit PCB
Parts:
- removed the D2 at (11.4, -25.4)
- added D4: BZX585-B5V6.115, Diode_SMD:D_SOD-523, B.Cu at (39.4, -21.1)
- C1, C10, C11, C12, C13, C14, C15, C16, C17, C18, C19, C2, C3, C4, C5, C6, C7, C8, C9, D1, D2, D3, J2, L1, R1, R2, R3, R4, R5, R6, R7, U1, U2, U3: moved to B.Cu
- J1: value 505405-0670 -> 213226-0611; moved to B.Cu
- moved H1 119.8 mm to (-83.8, -35.1)
- moved H2 119.8 mm to (-114.3, -35.1)
- moved H3 119.8 mm to (-114.3, -14.7)
- moved H4 119.8 mm to (-83.8, -14.7)
- moved C15 94.0 mm to (13.5, -3.92)
- moved U3 84.0 mm to (15.0, -8.37)
- moved R2 83.6 mm to (11.9, -13.2), turned to 180 degrees
- moved C10 82.1 mm to (10.5, -8.51), turned to -90 degrees
- moved C9 81.7 mm to (6.22, -3.43), turned to -90 degrees
- moved C7 81.1 mm to (3.30, -3.17), turned to -90 degrees
- moved C11 80.4 mm to (9.40, -3.30), turned to -90 degrees
- moved C2 77.1 mm to (0.38, -3.43), turned to -90 degrees
- moved C12 76.4 mm to (8.38, -10.8), turned to -90 degrees
- moved C18 73.9 mm to (42.3, 6.48), turned to -90 degrees
- moved C8 73.8 mm to (7.24, -8.51), turned to -90 degrees
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Connections:
- C11 pad 2: unconnected-(C11-Pad2) -> GND
- C2 pad 2: unconnected-(C2-Pad2) -> GND
- C7 pad 2: unconnected-(C7-Pad2) -> GND
- C9 pad 2: unconnected-(C9-Pad2) -> GND
- D3 pad 1: GND -> Net-(C15-Pad2)
- H1 pad 1: unconnected-(H1-Pad1) -> (no net)
- H2 pad 1: unconnected-(H2-Pad1) -> (no net)
- H3 pad 1: unconnected-(H3-Pad1) -> (no net)
- H4 pad 1: unconnected-(H4-Pad1) -> (no net)
- U1 pad 4: unconnected-(U1-Pad4) -> (no net)
- U1 pad 7: unconnected-(U1-Pad7) -> (no net)
- U2 pad 4: unconnected-(U2-Pad4) -> (no net)
Other:
- board size 40.1 x 30 mm -> 60 x 32 mm
- board text added: "5v3"
- board text added: "gnd"
- board text added: "sense current"
- board text added: "sense voltage"

Commit message: Edit PCB
Parts:
- removed H1, H2, H3, H4: M3, Mlab_Mechanical:MountingHole_3mm
- moved C13 77.3 mm to (2.34, -6.41)
- moved U2 71.0 mm to (5.66, -6.45)
- moved D2 68.3 mm to (6.48, -2.88)
- moved R1 65.5 mm to (13.6, -2.94), turned to 90 degrees
- moved C5 64.3 mm to (8.76, -2.94)
- moved C3 61.2 mm to (11.0, -2.94)
- moved D1 61.0 mm to (11.4, -6.60)
- moved R6 20.2 mm to (29.5, -2.63)
- moved R5 20.1 mm to (29.5, -6.19)
- moved C16 17.6 mm to (29.5, -10.1), turned to 90 degrees
- moved C17 16.7 mm to (32.1, -8.59), turned to 90 degrees
- moved J2 15.3 mm to (42.2, -23.1)
- moved J1 15.3 mm to (40.4, -8.26)
- moved J19 14.5 mm to (30.5, -24.5)
- moved C4 14.4 mm to (14.1, -28.0), turned to 180 degrees
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Connections:
- J1 pad 1: /5V3 -> GND
- J1 pad 2: /5V3 -> GND
- J1 pad 3: /SENSE_CURRENT -> /SENSE_VOLTAGE
- J1 pad 4: /SENSE_VOLTAGE -> /SENSE_CURRENT
- J1 pad 5: GND -> /5V3
- J1 pad 6: GND -> /5V3
- U3 pad 9: (no net) -> GND
Routing:
- net /SENSE_CURRENT: track 0.00 -> 39.2 mm, vias 0 -> 3
- net +3V3: track 0.00 -> 34.1 mm, vias 0 -> 2
- net /SENSE_VOLTAGE: track 0.00 -> 31.0 mm, vias 0 -> 3
- net /5V3: track 0.00 -> 30.9 mm
- net Net-(R5-Pad2): track 0.00 -> 24.4 mm, vias 0 -> 2
- net Net-(C15-Pad2): track 0.00 -> 6.40 mm
- net VCC: track 0.00 -> 4.81 mm
- net Net-(R2-Pad1): track 0.00 -> 3.47 mm
- net Net-(R7-Pad1): track 0.00 -> 3.25 mm
- net Net-(C14-Pad1): track 0.00 -> 2.90 mm
- net Net-(D1-Pad2): track 0.00 -> 2.74 mm
- net Net-(C15-Pad1): track 0.00 -> 2.12 mm
- net GND: vias 0 -> 101
- added copper zone on B.Cu, net /5V3
- added copper zone on B.Cu, net Net-(C15-Pad2)
- added copper zone on B.Cu, net Net-(J18-Pad1)
- added copper zone on B.Cu, net VCC
- added copper zone on F.Cu, net VCC
Other:
- board size 60 x 32 mm -> 45 x 30 mm
- board text removed: "5v3"
- board text removed: "gnd"
- board text removed: "sense current"
- board text removed: "sense voltage"

Commit message: Edit PCB
Parts:
- moved C8 0.51 mm to (4.57, -11.9)
- moved C7 0.46 mm to (7.11, -11.9)
- moved C9 0.46 mm to (2.03, -11.9)
- moved C2 0.46 mm to (9.65, -11.9)
- moved C10 0.41 mm to (12.2, -11.9)
Routing:
- net Net-(R5-Pad2): track 24.4 -> 23.9 mm
Changed lines of the file:
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@@
   )
   (footprint "Resistor_SMD:R_1206_3216Metric" (layer "B.Cu")
-    (at 4.064 -11.9096 -90)
+    (at 4.572 -11.9096 -90)
     (descr "Resistor SMD 1206 (3216 Metric), square (rectangular) end terminal, IPC_7351 nominal, (Body size source: http://www.tortai-tech.com/upload/download/2011102023233369053.pdf), generated with kicad-footprint-generator")
     (tags "resistor")
@@
   )
   (footprint "Resistor_SMD:R_1206_3216Metric" (layer "B.Cu")
-    (at 1.5748 -11.9096 -90)
+    (at 2.032 -11.9096 -90)
     (descr "Resistor SMD 1206 (3216 Metric), square (rectangular) end terminal, IPC_7351 nominal, (Body size source: http://www.tortai-tech.com/upload/download/2011102023233369053.pdf), generated with kicad-footprint-generator")
     (tags "resistor")
@@
   )
   (footprint "Resistor_SMD:R_1206_3216Metric" (layer "B.Cu")
-    (at 6.6548 -11.9096 -90)
+    (at 7.112 -11.9096 -90)
     (descr "Resistor SMD 1206 (3216 Metric), square (rectangular) end terminal, IPC_7351 nominal, (Body size source: http://www.tortai-tech.com/upload/download/2011102023233369053.pdf), generated with kicad-footprint-generator")
     (tags "resistor")
@@
   )
   (footprint "Resistor_SMD:R_1206_3216Metric" (layer "B.Cu")
-    (at 11.7856 -11.8648 -90)
+    (at 12.192 -11.8648 -90)
     (descr "Resistor SMD 1206 (3216 Metric), square (rectangular) end terminal, IPC_7351 nominal, (Body size source: http://www.tortai-tech.com/upload/download/2011102023233369053.pdf), generated with kicad-footprint-generator")
     (tags "resistor")
@@
   )
   (footprint "Resistor_SMD:R_1206_3216Metric" (layer "B.Cu")
-    (at 9.1948 -11.8588 -90)
+    (at 9.652 -11.8588 -90)
     (descr "Resistor SMD 1206 (3216 Metric), square (rectangular) end terminal, IPC_7351 nominal, (Body size source: http://www.tortai-tech.com/upload/download/2011102023233369053.pdf), generated with kicad-footprint-generator")
     (tags "resistor")
@@
   (via (at 25.908 -22.86) (size 0.8) (drill 0.4) (layers "F.Cu" "B.Cu") (free) (net 1))
   (via (at 2.286 -8.89) (size 0.8) (drill 0.4) (layers "F.Cu" "B.Cu") (free) (net 1))
-  (via (at 11.176 -29.21) (size 0.8) (drill 0.4) (layers "F.Cu" "B.Cu") (free) (net 1))
+  (via (at 11.176 -28.956) (size 0.8) (drill 0.4) (layers "F.Cu" "B.Cu") (free) (net 1))
   (via (at 34.036 -5.842) (size 0.8) (drill 0.4) (layers "F.Cu" "B.Cu") (free) (net 1))
   (via (at 35.306 -25.908) (size 0.8) (drill 0.4) (layers "F.Cu" "B.Cu") (free) (net 1))
@@
   (segment (start 15.116 -17.402) (end 16.383 -18.669) (width 0.4) (layer "B.Cu") (net 12))
   (segment (start 15.116 -16.764) (end 15.116 -17.402) (width 0.4) (layer "B.Cu") (net 12))
-  (segment (start 30.099 -15.621) (end 30.099 -5.08) (width 0.4) (layer "F.Cu") (net 13))
+  (segment (start 28.956 -15.621) (end 30.099 -14.478) (width 0.4) (layer "F.Cu") (net 13))
+  (segment (start 30.099 -14.478) (end 30.099 -5.08) (width 0.4) (layer "F.Cu") (net 13))
   (segment (start 30.099 -5.08) (end 29.464 -4.445) (width 0.4) (layer "F.Cu") (net 13))
-  (segment (start 21.59 -16.764) (end 28.956 -16.764) (width 0.4) (layer "F.Cu") (net 13))
-  (segment (start 28.956 -16.764) (end 30.099 -15.621) (width 0.4) (layer "F.Cu") (net 13))
+  (segment (start 21.59 -16.764) (end 21.59 -16.51) (width 0.4) (layer "F.Cu") (net 13))
+  (segment (start 21.59 -16.51) (end 22.479 -15.621) (width 0.4) (layer "F.Cu") (net 13))
+  (segment (start 22.479 -15.621) (end 28.956 -15.621) (width 0.4) (layer "F.Cu") (net 13))
   (via (at 29.464 -4.445) (size 0.8) (drill 0.4) (layers "F.Cu" "B.Cu") (net 13))
   (via (at 21.59 -16.764) (size 0.8) (drill 0.4) (layers "F.Cu" "B.Cu") (net 13))
@@
     (polygon
       (pts
-        (xy 30.48 -16.891)
+        (xy 30.48 -16.764)
         (xy 13.208 -16.764)
-        (xy 13.208 -22.098)
-        (xy 30.48 -22.098)
+        (xy 13.208 -21.844)
+        (xy 30.48 -21.844)
       )
     )
@@
         (xy 13.8684 -13.9192)
         (xy 12.5476 -12.5984)
-        (xy 0.7112 -12.5984)
-        (xy 0.7112 -13.9192)
+        (xy 1.143 -12.5984)
+        (xy 1.143 -14.097)
         (xy 1.7272 -14.9352)
         (xy 4.9784 -14.9352)
